File: BNC Shield +:-0.1-0.8.brd (EAGLE design)
At the start: 53.3 x 57.6 mm, 21 parts, among them IC2 TL072D, U1 ARDUINOR3-DIMENSION, X4 1-227161-0

Commit message: push
Parts:
- removed X1, X2, X3: (no value), con-rib:SH5-2
- added JP1: (no value), jumper:JP2
- added JP2, JP3, JP4, JP5, JP6, JP7: (no value), jumper:JP1
- added JP8: (no value), jumper:JP4Q
- U$1: value TC1121COA -> ADM660
- moved R6 33.8 mm to (31.2, 22.6)
- moved R7 22.3 mm to (31.2, 26.9)
- moved C3 21.2 mm to (21.3, 22.6)
- moved R4 19.3 mm to (41.4, 26.7)
- moved R11 16.2 mm to (25.1, 19.6)
- moved U$1 16.0 mm to (37.1, 16.0)
- moved R5 14.9 mm to (45.0, 31.5)
- moved R8 10.1 mm to (22.9, 40.9)
- moved X4 8.13 mm to (33.8, 49.5)
- moved IC2 7.18 mm to (34.3, 38.4), turned to 180 degrees
- moved R3 4.75 mm to (22.1, 47.0)
Connections:
- removed net N$10: C3.1, IC2.7, R11.2, R6.1, R7.1, R8.1
- new net N$13: JP8.2, U1.A0
- new net N$14: JP8.4, U1.A1
- new net N$15: JP8.6, U1.A2
- new net N$16: JP8.8, U1.A3
- new net TO_ARDUINO: C3.1, IC2.7, JP8.1, JP8.3, JP8.5, JP8.7, R11.2, R6.1, R7.1, R8.1
- net N$11: now also JP5.1, JP6.1, JP7.1; no longer X1.4, X2.4, X3.4
- net N$2: now also JP2.1; no longer X1.2
- net N$3: now also JP3.1; no longer X2.2
- net N$4: now also JP4.1; no longer X3.2
- net N$6: now also JP2.2, JP3.2, JP4.2; no longer X1.1, X2.1, X3.1
- net N$7: now also JP5.2; no longer X3.3
- net N$8: now also JP6.2; no longer X2.3
- net N$9: now also JP7.2; no longer X1.3

Commit message: push
Parts:
- added C4, C6: 100ufX6.3v, adafruit:153CLV-0605
- added C5, C7: 0.1uf, adafruit:C0603
- moved R3 21.3 mm to (30.5, 27.4), turned to 90 degrees
- moved C2 21.0 mm to (28.7, 36.3), turned to 270 degrees
- moved R8 20.3 mm to (38.1, 27.4), turned to 270 degrees
- moved C1 17.4 mm to (26.2, 36.3), turned to 270 degrees
- moved R10 15.2 mm to (33.0, 27.4), turned to 90 degrees
- moved JP7 15.0 mm to (26.7, 3.81)
- moved R9 14.4 mm to (23.6, 36.3), turned to 270 degrees
- moved JP6 12.8 mm to (24.4, 3.81)
- moved JP5 10.9 mm to (21.8, 3.56)
- moved R11 7.88 mm to (25.4, 27.4), turned to 270 degrees
- moved R2 7.61 mm to (21.1, 36.3), turned to 90 degrees
- moved R6 5.85 mm to (27.9, 27.4), turned to 270 degrees
- moved JP4 5.11 mm to (18.5, 4.06)
- moved C3 4.54 mm to (19.3, 26.7), turned to 90 degrees
- moved R5 4.44 mm to (43.2, 27.4), turned to 90 degrees
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Connections:
- new net -5V: C6.-, C7.2, U$1.5
- new net N$10: C4.+, U$1.2
- new net N$17: C4.-, U$1.4
- net GND: now also C5.1, C6.+, C7.1, U$1.3
- net VCC: now also C5.2, U$1.8
