File: BNC Shield +:-0.1-0.8.sch (EAGLE design)
At the start: 21 parts, among them IC2 TL072D, U1 ARDUINOR3-DIMENSION, X4 1-227161-0

Commit message: push
Parts:
- removed X1, X2, X3: (no value), con-rib:SH5-2
- added JP1: (no value), jumper:JP2E
- added JP2, JP3, JP4, JP5, JP6, JP7: (no value), jumper:JP1E
- added JP8: (no value), jumper:JP4Q
- U$1: value TC1121COA -> ADM660
Connections:
- removed net N$10: C3.1, IC2B.OUT, R11.2, R6.1, R7.1, R8.1
- new net N$13: JP8.2, U1.A0
- new net N$14: JP8.4, U1.A1
- new net N$15: JP8.6, U1.A2
- new net N$16: JP8.8, U1.A3
- new net TO_ARDUINO: C3.1, IC2B.OUT, JP8.1, JP8.3, JP8.5, JP8.7, R11.2, R6.1, R7.1, R8.1
- net N$11: now also JP5.1, JP6.1, JP7.1; no longer X1-2.2, X2-2.2, X3-2.2
- net N$2: now also JP2.1; no longer X1-1.2
- net N$3: now also JP3.1; no longer X2-1.2
- net N$4: now also JP4.1; no longer X3-1.2
- net N$6: now also JP2.2, JP3.2, JP4.2; no longer X1-1.1, X2-1.1, X3-1.1
- net N$7: now also JP5.2; no longer X3-2.1
- net N$8: now also JP6.2; no longer X2-2.1
- net N$9: now also JP7.2; no longer X1-2.1
Other:
- note added: "TO_ARDUINO"
Changed lines of the file:
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@@
 <parts>
 <part name="R1" library="resistor" deviceset="R-US_" device="R0603" value="100k"/>
-<part name="X1" library="con-rib" deviceset="SH5-2" device=""/>
 <part name="P+1" library="supply1" deviceset="VCC" device=""/>
-<part name="X2" library="con-rib" deviceset="SH5-2" device=""/>
-<part name="X3" library="con-rib" deviceset="SH5-2" device=""/>
 <part name="R2" library="resistor" deviceset="R-US_" device="R0603" value="100k"/>
 <part name="R3" library="resistor" deviceset="R-US_" device="R0603" value="1.91k"/>
@@
 <part name="X4" library="con-coax" deviceset="?227161*" device="1-" technology="-0"/>
 <part name="SUPPLY13" library="supply2" deviceset="GND" device=""/>
-<part name="U$1" library="tc1121" deviceset="TC1121" device="COA"/>
+<part name="U$1" library="tc1121" deviceset="TC1121" device="COA" value="ADM660"/>
+<part name="JP1" library="jumper" deviceset="JP2E" device=""/>
+<part name="JP2" library="jumper" deviceset="JP1E" device=""/>
+<part name="JP3" library="jumper" deviceset="JP1E" device=""/>
+<part name="JP4" library="jumper" deviceset="JP1E" device=""/>
+<part name="JP5" library="jumper" deviceset="JP1E" device=""/>
+<part name="JP6" library="jumper" deviceset="JP1E" device=""/>
+<part name="JP7" library="jumper" deviceset="JP1E" device=""/>
+<part name="JP8" library="jumper" deviceset="JP4Q" device=""/>
 </parts>
 <sheets>
@@
 <text x="-20.32" y="-35.56" size="1.778" layer="91">Jumper X2 for +/-0.414V input</text>
 <text x="-20.32" y="-38.1" size="1.778" layer="91">Jumper X3 for +/-0.1 input</text>
+<text x="-106.68" y="-10.16" size="1.778" layer="91" rot="R90">TO_ARDUINO</text>
+<text x="22.86" y="5.08" size="1.778" layer="91">TO_ARDUINO</text>
 </plain>
 <instances>
 <instance part="R1" gate="G$1" x="-53.34" y="22.86"/>
-<instance part="X1" gate="-1" x="-68.58" y="-17.78"/>
-<instance part="X1" gate="-2" x="-22.86" y="30.48" rot="R270"/>
 <instance part="P+1" gate="VCC" x="-10.16" y="17.78"/>
-<instance part="X2" gate="-1" x="-55.88" y="-17.78"/>
-<instance part="X2" gate="-2" x="-22.86" y="40.64" rot="R270"/>
-<instance part="X3" gate="-1" x="-43.18" y="-17.78"/>
-<instance part="X3" gate="-2" x="-22.86" y="50.8" rot="R270"/>
 <instance part="R2" gate="G$1" x="-53.34" y="5.08"/>
 <instance part="R3" gate="G$1" x="-63.5" y="-27.94" rot="R90"/>
@@
 <instance part="SUPPLY13" gate="GND" x="-109.22" y="15.24"/>
 <instance part="U$1" gate="G$1" x="-165.1" y="43.18"/>
+<instance part="JP1" gate="1" x="-177.8" y="60.96" rot="R90"/>
+<instance part="JP2" gate="A" x="-66.04" y="-17.78" rot="R90"/>
+<instance part="JP3" gate="A" x="-53.34" y="-17.78" rot="R90"/>
+<instance part="JP4" gate="A" x="-40.64" y="-17.78" rot="R90"/>
+<instance part="JP5" gate="A" x="-22.86" y="48.26"/>
+<instance part="JP6" gate="A" x="-22.86" y="38.1"/>
+<instance part="JP7" gate="A" x="-22.86" y="27.94"/>
+<instance part="JP8" gate="B" x="-119.38" y="2.54" rot="R90"/>
 </instances>
 <busses>
@@
 <segment>
 <wire x1="-63.5" y1="-17.78" x2="-63.5" y2="-22.86" width="0.1524" layer="91"/>
-<pinref part="X1" gate="-1" pin="2"/>
 <pinref part="R3" gate="G$1" pin="2"/>
+<pinref part="JP2" gate="A" pin="1"/>
 </segment>
 </net>
@@
 <segment>
 <wire x1="-50.8" y1="-17.78" x2="-50.8" y2="-22.86" width="0.1524" layer="91"/>
-<pinref part="X2" gate="-1" pin="2"/>
 <pinref part="R4" gate="G$1" pin="2"/>
+<pinref part="JP3" gate="A" pin="1"/>
 </segment>
 </net>
@@
 <segment>
 <wire x1="-38.1" y1="-17.78" x2="-38.1" y2="-22.86" width="0.1524" layer="91"/>
-<pinref part="X3" gate="-1" pin="2"/>
 <pinref part="R5" gate="G$1" pin="2"/>
+<pinref part="JP4" gate="A" pin="1"/>
 </segment>
 </net>
@@
 <junction x="-63.5" y="-10.16"/>
 <junction x="-50.8" y="-10.16"/>
-<pinref part="X3" gate="-1" pin="1"/>
-<pinref part="X1" gate="-1" pin="1"/>
-<pinref part="X2" gate="-1" pin="1"/>
 <pinref part="R9" gate="G$1" pin="2"/>
 <pinref part="R2" gate="G$1" pin="1"/>
 <pinref part="C2" gate="G$1" pin="1"/>
+<pinref part="JP2" gate="A" pin="2"/>
+<pinref part="JP3" gate="A" pin="2"/>
+<pinref part="JP4" gate="A" pin="2"/>
 </segment>
 </net>
@@
 <segment>
 <wire x1="-20.32" y1="45.72" x2="-15.24" y2="45.72" width="0.1524" layer="91"/>
-<pinref part="X3" gate="-2" pin="1"/>
 <pinref part="R6" gate="G$1" pin="2"/>
+<pinref part="JP5" gate="A" pin="2"/>
 </segment>
 </net>
@@
 <segment>
 <wire x1="-20.32" y1="35.56" x2="-15.24" y2="35.56" width="0.1524" layer="91"/>
-<pinref part="X2" gate="-2" pin="1"/>
 <pinref part="R7" gate="G$1" pin="2"/>
+<pinref part="JP6" gate="A" pin="2"/>
 </segment>
 </net>
@@
 <segment>
 <wire x1="-20.32" y1="25.4" x2="-15.24" y2="25.4" width="0.1524" layer="91"/>
-<pinref part="X1" gate="-2" pin="1"/>
 <pinref part="R8" gate="G$1" pin="2"/>
-</segment>
-</net>
-<net name="N$10" class="0">
+<pinref part="JP7" gate="A" pin="2"/>
+</segment>
+</net>
+<net name="TO_ARDUINO" class="0">
 <segment>
 <wire x1="-5.08" y1="45.72" x2="-2.54" y2="43.18" width="0.1524" layer="91"/>
@@
 <pinref part="IC2" gate="B" pin="OUT"/>
 </segment>
+<segment>
+<pinref part="JP8" gate="B" pin="7"/>
+<wire x1="-111.76" y1="7.62" x2="-109.22" y2="7.62" width="0.1524" layer="91"/>
+<wire x1="-109.22" y1="7.62" x2="-109.22" y2="5.08" width="0.1524" layer="91"/>
+<pinref part="JP8" gate="B" pin="5"/>
+<wire x1="-109.22" y1="5.08" x2="-109.22" y2="2.54" width="0.1524" layer="91"/>
+<wire x1="-109.22" y1="2.54" x2="-109.22" y2="0" width="0.1524" layer="91"/>
+<wire x1="-109.22" y1="0" x2="-109.22" y2="-5.08" width="0.1524" layer="91"/>
+<wire x1="-111.76" y1="5.08" x2="-109.22" y2="5.08" width="0.1524" layer="91"/>
+<pinref part="JP8" gate="B" pin="3"/>
+<wire x1="-111.76" y1="2.54" x2="-109.22" y2="2.54" width="0.1524" layer="91"/>
+<pinref part="JP8" gate="B" pin="1"/>
+<wire x1="-111.76" y1="0" x2="-109.22" y2="0" width="0.1524" layer="91"/>
+</segment>
 </net>
 <net name="N$11" class="0">
@@
 <junction x="-27.94" y="25.4"/>
 <junction x="-27.94" y="35.56"/>
-<pinref part="X3" gate="-2" pin="2"/>
-<pinref part="X2" gate="-2" pin="2"/>
-<pinref part="X1" gate="-2" pin="2"/>
 <pinref part="R10" gate="G$1" pin="2"/>
 <pinref part="IC2" gate="B" pin="-IN"/>
+<pinref part="JP5" gate="A" pin="1"/>
+<pinref part="JP6" gate="A" pin="1"/>
+<pinref part="JP7" gate="A" pin="1"/>
 </segment>
 </net>
@@
 </segment>
 </net>
+<net name="N$13" class="0">
+<segment>
+<pinref part="U1" gate="G$1" pin="A0"/>
+<pinref part="JP8" gate="B" pin="2"/>
+<wire x1="-127" y1="0" x2="-134.62" y2="0" width="0.1524" layer="91"/>
+</segment>
+</net>
+<net name="N$14" class="0">
+<segment>
+<pinref part="U1" gate="G$1" pin="A1"/>
+<pinref part="JP8" gate="B" pin="4"/>
+<wire x1="-127" y1="2.54" x2="-134.62" y2="2.54" width="0.1524" layer="91"/>
+</segment>
+</net>
+<net name="N$15" class="0">
+<segment>
+<pinref part="U1" gate="G$1" pin="A2"/>
+<pinref part="JP8" gate="B" pin="6"/>
+<wire x1="-127" y1="5.08" x2="-134.62" y2="5.08" width="0.1524" layer="91"/>
+</segment>
+</net>
+<net name="N$16" class="0">
+<segment>
+<pinref part="U1" gate="G$1" pin="A3"/>
+<pinref part="JP8" gate="B" pin="8"/>
+<wire x1="-127" y1="7.62" x2="-134.62" y2="7.62" width="0.1524" layer="91"/>
+</segment>
+</net>

Commit message: push
Parts:
- added C4, C6: 100ufX6.3v, adafruit:CPOL-US153CLV-0605
- added C5, C7: 0.1uf, adafruit:C-USC0603
Connections:
- new net -5V: C6.-, C7.2, U$1.VOUT
- new net N$10: C4.+, U$1.CAP+
- new net N$17: C4.-, U$1.CAP-
- net GND: now also C5.1, C6.+, C7.1, U$1.GND
- net VCC: now also C5.2, U$1.VIN
Changed lines of the file:
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@@
 <part name="JP7" library="jumper" deviceset="JP1E" device=""/>
 <part name="JP8" library="jumper" deviceset="JP4Q" device=""/>
+<part name="C4" library="adafruit" deviceset="CPOL-US" device="153CLV-0605" value="100ufX6.3v"/>
+<part name="SUPPLY1" library="supply2" deviceset="GND" device=""/>
+<part name="P+3" library="supply1" deviceset="VCC" device=""/>
+<part name="C5" library="adafruit" deviceset="C-US" device="C0603" value="0.1uf"/>
+<part name="SUPPLY2" library="supply2" deviceset="GND" device=""/>
+<part name="SUPPLY8" library="supply2" deviceset="-5V" device=""/>
+<part name="SUPPLY9" library="supply2" deviceset="-5V" device=""/>
+<part name="C6" library="adafruit" deviceset="CPOL-US" device="153CLV-0605" value="100ufX6.3v"/>
+<part name="C7" library="adafruit" deviceset="C-US" device="C0603" value="0.1uf"/>
+<part name="SUPPLY14" library="supply2" deviceset="GND" device=""/>
+<part name="SUPPLY15" library="supply2" deviceset="GND" device=""/>
 </parts>
 <sheets>
@@
 <instance part="JP7" gate="A" x="-22.86" y="27.94"/>
 <instance part="JP8" gate="B" x="-119.38" y="2.54" rot="R90"/>
+<instance part="C4" gate="G$1" x="-193.04" y="40.64"/>
+<instance part="SUPPLY1" gate="GND" x="-182.88" y="40.64" rot="R270"/>
+<instance part="P+3" gate="VCC" x="-132.08" y="45.72" rot="R270"/>
+<instance part="C5" gate="G$1" x="-144.78" y="53.34"/>
+<instance part="SUPPLY2" gate="GND" x="-144.78" y="60.96" rot="R180"/>
+<instance part="SUPPLY8" gate="-5V" x="-129.54" y="38.1" rot="R90"/>
+<instance part="SUPPLY9" gate="-5V" x="-10.16" y="-7.62"/>
+<instance part="C6" gate="G$1" x="-147.32" y="30.48" rot="R180"/>
+<instance part="C7" gate="G$1" x="-137.16" y="30.48" rot="R180"/>
+<instance part="SUPPLY14" gate="GND" x="-137.16" y="25.4"/>
+<instance part="SUPPLY15" gate="GND" x="-147.32" y="25.4"/>
 </instances>
 <busses>
@@
 <pinref part="SUPPLY13" gate="GND" pin="GND"/>
 <wire x1="-109.22" y1="17.78" x2="-109.22" y2="22.86" width="0.1524" layer="91"/>
+</segment>
+<segment>
+<pinref part="U$1" gate="G$1" pin="GND"/>
+<pinref part="SUPPLY1" gate="GND" pin="GND"/>
+</segment>
+<segment>
+<pinref part="C7" gate="G$1" pin="1"/>
+<pinref part="SUPPLY14" gate="GND" pin="GND"/>
+</segment>
+<segment>
+<pinref part="C6" gate="G$1" pin="+"/>
+<pinref part="SUPPLY15" gate="GND" pin="GND"/>
+</segment>
+<segment>
+<pinref part="SUPPLY2" gate="GND" pin="GND"/>
+<pinref part="C5" gate="G$1" pin="1"/>
+<wire x1="-144.78" y1="58.42" x2="-144.78" y2="55.88" width="0.1524" layer="91"/>
 </segment>
 </net>
@@
 <pinref part="P+4" gate="VCC" pin="VCC"/>
 <wire x1="-132.08" y1="-20.32" x2="-134.62" y2="-12.7" width="0.1524" layer="91"/>
+</segment>
+<segment>
+<pinref part="U$1" gate="G$1" pin="VIN"/>
+<pinref part="P+3" gate="VCC" pin="VCC"/>
+<wire x1="-134.62" y1="45.72" x2="-144.78" y2="45.72" width="0.1524" layer="91"/>
+<pinref part="C5" gate="G$1" pin="2"/>
+<wire x1="-144.78" y1="45.72" x2="-149.86" y2="45.72" width="0.1524" layer="91"/>
+<wire x1="-144.78" y1="48.26" x2="-144.78" y2="45.72" width="0.1524" layer="91"/>
 </segment>
 </net>
@@
 </segment>
 </net>
+<net name="N$10" class="0">
+<segment>
+<pinref part="U$1" gate="G$1" pin="CAP+"/>
+<pinref part="C4" gate="G$1" pin="+"/>
+<wire x1="-180.34" y1="43.18" x2="-193.04" y2="43.18" width="0.1524" layer="91"/>
+</segment>
+</net>
+<net name="N$17" class="0">
+<segment>
+<pinref part="U$1" gate="G$1" pin="CAP-"/>
+<wire x1="-180.34" y1="38.1" x2="-180.34" y2="35.56" width="0.1524" layer="91"/>
+<pinref part="C4" gate="G$1" pin="-"/>
+<wire x1="-180.34" y1="35.56" x2="-193.04" y2="35.56" width="0.1524" layer="91"/>
+</segment>
+</net>
+<net name="-5V" class="0">
+<segment>
+<pinref part="U$1" gate="G$1" pin="VOUT"/>
+<pinref part="SUPPLY8" gate="-5V" pin="-5V"/>
+<wire x1="-132.08" y1="38.1" x2="-137.16" y2="38.1" width="0.1524" layer="91"/>
+<pinref part="C6" gate="G$1" pin="-"/>
+<wire x1="-137.16" y1="38.1" x2="-147.32" y2="38.1" width="0.1524" layer="91"/>
+<wire x1="-147.32" y1="38.1" x2="-149.86" y2="38.1" width="0.1524" layer="91"/>
+<wire x1="-147.32" y1="38.1" x2="-147.32" y2="35.56" width="0.1524" layer="91"/>
+<pinref part="C7" gate="G$1" pin="2"/>
+<wire x1="-137.16" y1="38.1" x2="-137.16" y2="35.56" width="0.1524" layer="91"/>
+</segment>
+</net>
