File: BNC Shield 0.1-0.8 SMD.sch (EAGLE design)
At the start: 30 parts, among them IC2 TL072D, U1 ARDUINOR3-DIMENSION, X4 1-227161-0

Commit message: push to github
Parts:
- removed C6: 100ufX6.3v, adafruit:CPOL-US153CLV-0605
- removed C7: 0.1uf, adafruit:C-USC0603
- removed JP3, JP4, JP5, JP6, JP7: (no value), jumper:JP1E
- removed U$1: ADM660, tc1121:TC1121COA
- added C10, C9: 1u, dp_devices:CAPACITOR_NPOL-0603
- added C8: 100ufX6.3v, adafruit:CPOL-US153CLV-0605
- added IC1: TPS60400DBV, SparkysWidgets:TPS60400DBV
- added JP9: (no value), jumper:JP4Q
- added LED1, LED2: (no value), adafruit:LEDCHIP-LED0603
- added R12, R13: 150, resistor:R-US_R0603
- added R14: 205, resistor:R-US_R0603
- added R15: 51k, resistor:R-US_R0603
- added U$2, U$3, U$4, U$5: FIDUCIAL, adafruit:FIDUCIAL
- C3: value 100uF -> 1u; device resistor:C-USC0603 -> dp_devices:CAPACITOR_NPOL-0603
- C4: value 100ufX6.3v -> 0.1uf; device adafruit:CPOL-US153CLV-0605 -> dp_devices:CAPACITOR_NPOL-0603
- C5: device adafruit:C-USC0603 -> dp_devices:CAPACITOR_NPOL-0603
- JP2: device jumper:JP1E -> jumper:JP8QE
- JP8: device jumper:JP4Q -> jumper:JP6Q
- R5: value 205 -> 400
- R6: value 490k -> 110k
- R7: value 110k -> 240k
- R8: value 50.5k -> 490k
Connections:
- new net N$18: LED2.C, R12.1
- new net N$19: LED1.A, R13.2
- new net N$21: JP8.10, U1.A4/SDA
- new net N$22: C3.1, IC1.CFLY-
- new net N$23: C3.2, IC1.CFLY+
- new net N$24: JP9.5, U1.D3
- new net N$25: JP9.7, U1.D2
- new net N$26: JP8.12, U1.A5/SCL
- new net N$27: JP2-4.1, R14.2
- new net N$28: JP2-5.1, R15.2
- new net ONEWIRE_DATA: JP1.2, JP9.2, JP9.4, JP9.6, JP9.8
- net -5V: now also C10.2, C5.1, IC1.OUT, IC2P.V-, R12.2; no longer C6.-, C7.2, U$1.VOUT
- net GND: now also C10.1, C4.2, C5.2, C8.-, C9.2, IC1.GND, JP1.1, LED1.C, LED2.A, R14.1; no longer C3.2, C5.1, C6.+, C7.1, U$1.GND
- net N$10: now also JP9.1, U1.D5; no longer C4.+, U$1.CAP+
- net N$11: now also JP2-5.2, JP2-6.2, JP2-7.2, JP2-8.2; no longer JP5.1, JP6.1, JP7.1
- net N$17: now also JP9.3, U1.D4; no longer C4.-, U$1.CAP-
- net N$2: now also JP2-1.1; no longer JP2.1
- net N$3: now also JP2-2.1; no longer JP3.1
- net N$4: now also JP2-3.1; no longer JP4.1
- net N$6: now also JP2-1.2, JP2-2.2, JP2-3.2, JP2-4.2; no longer JP2.2, JP3.2, JP4.2
- net N$7: now also JP2-6.1; no longer JP5.2
- net N$8: now also JP2-7.1; no longer JP6.2
- net N$9: now also JP2-8.1; no longer JP7.2
- net TO_ARDUINO: now also C8.+, JP8.11, JP8.9, R15.1; no longer C3.1
- net VCC: now also C4.1, C9.1, IC1.IN, IC2P.V+, JP1.3, R13.1; no longer C5.2, U$1.VIN
Other:
- note added: "ONEWIRE_DATA"
- note removed: "Jumper X1 for +/-0.8V input"
- note removed: "Jumper X2 for +/-0.414V input"
- note removed: "Jumper X3 for +/-0.1 input"
- moved on the sheet: R3, R4, R5
